Commit message: version 1.0.0

File: src/system_bringup/urdf/robot_base.urdf (robot description, URDF)
Before this commit: robot Shopping Cart Robot, 13 links, 12 joints
Links:
- removed link panel_link
- added link base_footprint
- added link camera_link, mass 0.0613007198991268; collision mesh filename=package://URDF_RobotDiploma/meshes/camera_link.STL; visual mesh filename=package://URDF_RobotDiploma/meshes/camera_link.STL
- link back_caster: mass 0.0153736904053634 -> 0.00259129992796193; geometry collision mesh filename=package://URDF_RobotDiploma/meshes/back_caster.STL; visual mesh filename=package://URDF_RobotDiploma/meshes/back_caster.STL
- link back_caster_wheel: mass 0.00261436300403997 -> 0.00382605152201998; geometry collision mesh filename=package://URDF_RobotDiploma/meshes/back_caster_wheel.STL; visual mesh filename=package://URDF_RobotDiploma/meshes/back_caster_wheel.STL
- link base_link: mass 4.90310056097342 -> 7.4355; geometry collision mesh filename=package://URDF_RobotDiploma/meshes/base_link.STL; visual mesh filename=package://URDF_RobotDiploma/meshes/base_link.STL
- link front_caster: mass 0.0107307157974003 -> 0.00259129992796221; geometry collision mesh filename=package://URDF_RobotDiploma/meshes/front_caster.STL; visual mesh filename=package://URDF_RobotDiploma/meshes/front_caster.STL
- link front_caster_wheel: mass 0.00725733761200358 -> 0.00382605152202009; geometry collision mesh filename=package://URDF_RobotDiploma/meshes/front_caster_wheel.STL; visual mesh filename=package://URDF_RobotDiploma/meshes/front_caster_wheel.STL
- link left_wheel: mass 0.0713374663725933 -> 0.533369044032681; geometry collision mesh filename=package://URDF_RobotDiploma/meshes/left_wheel.STL; visual mesh filename=package://URDF_RobotDiploma/meshes/left_wheel.STL
- link lidar_back_left: mass 0.0260070250802488 -> 0.10251; geometry collision mesh filename=package://URDF_RobotDiploma/meshes/lidar_back_left.STL; visual mesh filename=package://URDF_RobotDiploma/meshes/lidar_back_left.STL
- link lidar_back_right: mass 0.0260070238651023 -> 0.102513123915553; geometry collision mesh filename=package://URDF_RobotDiploma/meshes/lidar_back_right.STL; visual mesh filename=package://URDF_RobotDiploma/meshes/lidar_back_right.STL
- link lidar_front_left: mass 0.0260070151534254 -> 0.102513124786789; geometry collision mesh filename=package://URDF_RobotDiploma/meshes/lidar_front_left.STL; visual mesh filename=package://URDF_RobotDiploma/meshes/lidar_front_left.STL
- link lidar_front_right: mass 0.0260070168506664 -> 0.102513137152156; geometry collision mesh filename=package://URDF_RobotDiploma/meshes/lidar_front_right.STL; visual mesh filename=package://URDF_RobotDiploma/meshes/lidar_front_right.STL
- link right_wheel: mass 0.0713374663725935 -> 0.533369044032682; geometry collision mesh filename=package://URDF_RobotDiploma/meshes/right_wheel.STL; visual mesh filename=package://URDF_RobotDiploma/meshes/right_wheel.STL
- link top_link: mass 4.55501076764544 -> 0; geometry collision mesh filename=package://URDF_RobotDiploma/meshes/top_link.STL; visual mesh filename=package://URDF_RobotDiploma/meshes/top_link.STL
Joints:
- removed joint panellinkjoint
- added joint base_footprint_joint: type fixed, parent base_footprint, child base_link, origin xyz=0 0 0.05 rpy=0 0 0
- added joint camera_joint: type fixed, parent top_link, child camera_link, origin xyz=0.03246 -0.002 0.36 rpy=1.5708 0 1.5708, axis 0 0 0
- joint backcasterjoint: axis 0 0 -1 -> 0 0 1; origin xyz=-0.140000000000001 0 -0.0619999999999999 rpy=0 0 0 -> xyz=-0.12673 -0.0024611 -0.024392 rpy=0 0 0
- joint backcasterwheeljoint: axis -0.063897905647706 0 0.997956440759734 -> 0 0 -1; origin xyz=-0.0128973307994271 0.00984422969308141 -0.013 rpy=1.5707963267949 0 0 -> xyz=-0.012 -0.0104 -0.017111 rpy=1.5708 0 0
- joint frontcasterjoint: axis 0 0 -1 -> 0 0 1; origin xyz=0.14 0 -0.0620000000000001 rpy=0 0 0 -> xyz=0.128305917608629 3.08857392976591E-05 -0.024391789843072 rpy=0 0 0
- joint frontcasterwheeljoint: axis -0.063897905647706 0 0.997956440759734 -> 0 0 -1; origin xyz=-0.0128973307994271 0.00984422969308141 -0.013 rpy=1.5707963267949 0 0 -> xyz=-0.012 -0.0104 -0.017111 rpy=1.5708 0 0
- joint leftwheel: origin xyz=0.00656145183365686 0.166 -0.0500762565788667 rpy=1.5707963267949 0 0 -> xyz=0.00033999 0.194 0.013 rpy=1.5708 0 0
- joint lidar1: axis 0 0 1 -> 0 0 0; origin xyz=0.136139650045003 -0.0861403499550002 -0.0264 rpy=0 0 0 -> xyz=0.143897827735137 -0.1185 0.0232921469155075 rpy=0 0 0; type continuous -> fixed
- joint lidar2: axis 0 0 1 -> 0 0 0; origin xyz=0.136139650045006 0.0861403499549938 -0.0264 rpy=0 0 0 -> xyz=0.1439 0.1185 0.023292 rpy=0 0 0; type continuous -> fixed
- joint lidar3: origin xyz=-0.136140349954999 0.0861396500450031 -0.0264 rpy=0 0 0 -> xyz=-0.143102172264863 0.1185 0.0232921469155075 rpy=0 0 0; type continuous -> fixed
- joint lidar4: axis 0 0 1 -> 0 0 0; origin xyz=-0.13613965004501 -0.0861403499549971 -0.0264000000000001 rpy=0 0 0 -> xyz=-0.1431 -0.1185 0.023292 rpy=0 0 0; type continuous -> fixed
- joint rightwheel: origin xyz=0.00656145183365686 -0.166 -0.0500762565788665 rpy=1.5707963267949 0 0 -> xyz=0.00045567 -0.194 0.013 rpy=1.5708 0 0
- joint toplinkjoint: origin xyz=-0.000243515949483131 0 0 rpy=0 0 0 -> xyz=0.11794 0 0.065 rpy=0 0 0

Commit message: update 1.1.2

File: src/system_bringup/urdf/robot_base.urdf (robot description, URDF)
Before this commit: robot URDF_RobotDiploma, 14 links, 13 joints
Links:
- removed link back_caster_wheel
- removed link base_footprint
- removed link base_link
- removed link front_caster_wheel
- added link custom_base_footprint
- added link custom_base_link; collision box size=0.4 0.44 0.2; visual mesh filename=package://URDF_RobotDiploma/meshes/base_link.STL
- link back_caster: mass 0.00259129992796193 -> None; geometry visual mesh filename=package://URDF_RobotDiploma/meshes/back_caster.STL
- link camera_link: mass 0.0613007198991268 -> None; geometry visual mesh filename=package://URDF_RobotDiploma/meshes/camera_link.STL
- link front_caster: mass 0.00259129992796221 -> None; geometry visual mesh filename=package://URDF_RobotDiploma/meshes/front_caster.STL
- link left_wheel: mass 0.533369044032681 -> None; geometry collision cylinder length=0.04 radius=0.067; visual mesh filename=package://URDF_RobotDiploma/meshes/left_wheel.STL
- link lidar_back_left: mass 0.10251 -> None; geometry visual mesh filename=package://URDF_RobotDiploma/meshes/lidar_back_left.STL
- link lidar_back_right: mass 0.102513123915553 -> None; geometry visual mesh filename=package://URDF_RobotDiploma/meshes/lidar_back_right.STL
- link lidar_front_left: mass 0.102513124786789 -> None; geometry visual mesh filename=package://URDF_RobotDiploma/meshes/lidar_front_left.STL
- link lidar_front_right: mass 0.102513137152156 -> None; geometry visual mesh filename=package://URDF_RobotDiploma/meshes/lidar_front_right.STL
- link right_wheel: mass 0.533369044032682 -> None; geometry collision cylinder length=0.04 radius=0.067; visual mesh filename=package://URDF_RobotDiploma/meshes/right_wheel.STL
- link top_link: mass 0 -> None; geometry visual mesh filename=package://URDF_RobotDiploma/meshes/top_link.STL
Joints:
- removed joint backcasterwheeljoint
- removed joint frontcasterwheeljoint
- joint backcasterjoint: axis 0 0 1 -> (none); limit effort=10 velocity=10 -> (none); origin xyz=-0.12673 -0.0024611 -0.024392 rpy=0 0 0 -> xyz=-0.1267 0 -0.0243 rpy=0 0 0; parent base_link -> custom_base_link; type continuous -> fixed
- joint base_footprint_joint: child base_link -> custom_base_link; parent base_footprint -> custom_base_footprint
- joint camera_joint: axis 0 0 0 -> (none); origin xyz=0.03246 -0.002 0.36 rpy=1.5708 0 1.5708 -> xyz=0.0324 -0.002 0.36 rpy=1.5708 0 1.5708
- joint frontcasterjoint: axis 0 0 1 -> (none); limit effort=10 velocity=10 -> (none); origin xyz=0.128305917608629 3.08857392976591E-05 -0.024391789843072 rpy=0 0 0 -> xyz=0.1283 0 -0.0243 rpy=0 0 0; parent base_link -> custom_base_link; type continuous -> fixed
- joint leftwheel: limit effort=10 velocity=10 -> (none); parent base_link -> custom_base_link
- joint lidar1: axis 0 0 0 -> (none); origin xyz=0.143897827735137 -0.1185 0.0232921469155075 rpy=0 0 0 -> xyz=0.1438 -0.1185 0.0232 rpy=0 0 0; parent base_link -> custom_base_link
- joint lidar2: axis 0 0 0 -> (none); origin xyz=0.1439 0.1185 0.023292 rpy=0 0 0 -> xyz=0.1439 0.1185 0.0232 rpy=0 0 0; parent base_link -> custom_base_link
- joint lidar3: axis 0 0 1 -> (none); origin xyz=-0.143102172264863 0.1185 0.0232921469155075 rpy=0 0 0 -> xyz=-0.1431 0.1185 0.0232 rpy=0 0 0; parent base_link -> custom_base_link
- joint lidar4: axis 0 0 0 -> (none); origin xyz=-0.1431 -0.1185 0.023292 rpy=0 0 0 -> xyz=-0.1431 -0.1185 0.0232 rpy=0 0 0; parent base_link -> custom_base_link
- joint rightwheel: limit effort=10 velocity=10 -> (none); parent base_link -> custom_base_link
- joint toplinkjoint: axis 0 0 0 -> (none); origin xyz=0.11794 0 0.065 rpy=0 0 0 -> xyz=0.1179 0 0.065 rpy=0 0 0; parent base_link -> custom_base_link

Commit message: version 1.1.3

File: src/system_bringup/urdf/robot_base.urdf (robot description, URDF)
Before this commit: robot URDF_RobotDiploma, 12 links, 11 joints
Joints:
- joint lidar1: origin xyz=0.1438 -0.1185 0.0232 rpy=0 0 0 -> xyz=0.1438 -0.1185 0.0232 rpy=0 3.14159 0
- joint lidar2: origin xyz=0.1439 0.1185 0.0232 rpy=0 0 0 -> xyz=0.1439 0.1185 0.0232 rpy=0 3.14159 0

Commit message: version 2.0.0

File: src/system_bringup/urdf/robot_base.urdf (robot description, URDF)
Before this commit: robot URDF_RobotDiploma, 12 links, 11 joints
Joints:
- joint lidar1: origin xyz=0.1438 -0.1185 0.0232 rpy=0 3.14159 0 -> xyz=0.1438 -0.1185 0.0232 rpy=0 0 3.14159
- joint lidar2: origin xyz=0.1439 0.1185 0.0232 rpy=0 3.14159 0 -> xyz=0.1439 0.1185 0.0232 rpy=0 0 3.14159

Commit message: version 2.0.1

File: src/system_bringup/urdf/robot_base.urdf (robot description, URDF)
Before this commit: robot URDF_RobotDiploma, 12 links, 11 joints
Links:
- link back_caster: geometry visual mesh filename=package://system_bringup/meshes/back_caster.STL
- link camera_link: geometry visual mesh filename=package://system_bringup/meshes/camera_link.STL
- link custom_base_link: geometry collision box size=0.4 0.44 0.2; visual mesh filename=package://system_bringup/meshes/base_link.STL
- link front_caster: geometry visual mesh filename=package://system_bringup/meshes/front_caster.STL
- link left_wheel: geometry collision cylinder length=0.04 radius=0.067; visual mesh filename=package://system_bringup/meshes/left_wheel.STL
- link lidar_back_left: geometry visual mesh filename=package://system_bringup/meshes/lidar_back_left.STL
- link lidar_back_right: geometry visual mesh filename=package://system_bringup/meshes/lidar_back_right.STL
- link lidar_front_left: geometry visual mesh filename=package://system_bringup/meshes/lidar_front_left.STL
- link lidar_front_right: geometry visual mesh filename=package://system_bringup/meshes/lidar_front_right.STL
- link right_wheel: geometry collision cylinder length=0.04 radius=0.067; visual mesh filename=package://system_bringup/meshes/right_wheel.STL
- link top_link: geometry visual mesh filename=package://system_bringup/meshes/top_link.STL
